Commit message: adds a simple pendulum
git-svn-id: https://atrias.googlecode.com/svn/trunk@713 a504bc44-2baa-4cb8-4136-ba805e94d278

File: drl-sim/atrias/robots/boomTest.urdf.xacro (robot description, xacro)
@@ -16,4 +16,5 @@
 	<property name="upright_length" value="1" />
 	<property name="boom_length" value="1" />
+	<property name="pendulum_length" value="0.9" />
 	<property name="spring_stiffness" value="500" />
 	<property name="leg_seg_damping" value="0" />
@@ -61,5 +62,5 @@
 		<!--				 Boom					-->
 		<!--#########################################################################-->
-		<joint name="uprigh_boom_joint" type="continuous">
+		<joint name="upright_boom_joint" type="fixed">
 			<axis xyz="0 0 1" />
 			<!-- anchor xyz="0 0 0" / -->
@@ -71,5 +72,4 @@
 			<inertial>
 				<mass value="0.68292"/>
-				<!--mass value="9999999999" /-->
 				<origin xyz="${boom_length/2} 0 0" rpy="0 0 0" />
 				<inertia ixx="0.02116" ixy="0" ixz="0"
@@ -93,4 +93,37 @@
 			<material>Gazebo/Red</material>
 		</gazebo>
+		<!--#########################################################################-->
+		<!--				 Pendulum                                    -->
+		<!--#########################################################################-->
+		<joint name="pendulum_joint" type="continuous">
+			<axis xyz="1 0 0" />
+			<origin xyz="${boom_length} 0 0" rpy="${M_PI/18} 0 0" />
+			<parent link="boom_link" />
+			<child link="pendulum_link"/>
+		</joint>
+		<link name="pendulum_link">
+			<inertial>
+				<mass value="1"/>
+				<origin xyz="0 0 ${-pendulum_length/2}" rpy="0 0 0" />
+				<inertia ixx="0.245" ixy="0" ixz="0"
+				         iyy="0" iyz="0"
+				         izz="0" />
+			</inertial>
+			<visual>
+				<origin xyz="0 0 ${-pendulum_length/2}" rpy="0 0 0" />
+				<geometry>
+				  <cylinder length="${pendulum_length}" radius="${leg_segment_radius}" />
+				</geometry>
+			</visual>
+			<collision>
+				<origin xyz="0 0 ${-pendulum_length/2}" rpy="0 0 0" />
+				<geometry>
+					<cylinder length="${pendulum_length}" radius="${leg_segment_radius}" />
+				</geometry>
+			</collision>
+		</link>
+		<gazebo reference="pendulum_link">
+			<material>Gazebo/Red</material>
+		</gazebo>
 	</xacro:macro>
 </robot>

Commit message: The correct x-axis moment of inertia now causes a 2-second period of oscillation. Note that y- and z-axis moments of inertia needed to be set to an arbitrary non-zero value or else the period was too high.
git-svn-id: https://atrias.googlecode.com/svn/trunk@714 a504bc44-2baa-4cb8-4136-ba805e94d278

File: drl-sim/atrias/robots/boomTest.urdf.xacro (robot description, xacro)
@@ -98,5 +98,5 @@
 		<joint name="pendulum_joint" type="continuous">
 			<axis xyz="1 0 0" />
-			<origin xyz="${boom_length} 0 0" rpy="${M_PI/18} 0 0" />
+			<origin xyz="${boom_length} 0 0" rpy="${M_PI/18/5} 0 0" />
 			<parent link="boom_link" />
 			<child link="pendulum_link"/>
@@ -107,6 +107,6 @@
 				<origin xyz="0 0 ${-pendulum_length/2}" rpy="0 0 0" />
 				<inertia ixx="0.245" ixy="0" ixz="0"
-				         iyy="0" iyz="0"
-				         izz="0" />
+				         iyy="1" iyz="0"
+				         izz="1" />
 			</inertial>
 			<visual>

Commit message: Add a spring and a controller that publishes a 3D position topic. The predicted and actual period of oscillation is now T=1.5s.
git-svn-id: https://atrias.googlecode.com/svn/trunk@737 a504bc44-2baa-4cb8-4136-ba805e94d278

File: drl-sim/atrias/robots/boomTest.urdf.xacro (robot description, xacro)
@@ -17,5 +17,5 @@
 	<property name="boom_length" value="1" />
 	<property name="pendulum_length" value="0.9" />
-	<property name="spring_stiffness" value="500" />
+	<property name="spring_stiffness" value="3.5" />
 	<property name="leg_seg_damping" value="0" />
 	<!-- Initial Condition -->
@@ -31,4 +31,5 @@
 		<joint name="world_upright_joint" type="fixed">
 			<!-- anchor xyz="0 0 0" / -->
+			<axis xyz="0 0 1" rpy="0 0 0" />
 			<origin xyz="0 0 0" rpy="0 0 0" />
 			<parent link="world" />
@@ -92,4 +93,5 @@
 		<gazebo reference="boom_link">
 			<material>Gazebo/Red</material>
+			<static>true</static>
 		</gazebo>
 		<!--#########################################################################-->
@@ -97,6 +99,6 @@
 		<!--#########################################################################-->
 		<joint name="pendulum_joint" type="continuous">
-			<axis xyz="1 0 0" />
-			<origin xyz="${boom_length} 0 0" rpy="${M_PI/18/5} 0 0" />
+			<axis xyz="0 1 0" />
+			<origin xyz="${boom_length} 0 0" rpy="0 ${M_PI/18/5} 0" />
 			<parent link="boom_link" />
 			<child link="pendulum_link"/>
@@ -107,6 +109,6 @@
 				<origin xyz="0 0 ${-pendulum_length/2}" rpy="0 0 0" />
 				<inertia ixx="0.245" ixy="0" ixz="0"
-				         iyy="1" iyz="0"
-				         izz="1" />
+				         iyy="0.245" iyz="0"
+				         izz="0.245" />
 			</inertial>
 			<visual>
@@ -126,4 +128,26 @@
 			<material>Gazebo/Red</material>
 		</gazebo>
+		<gazebo>
+			<controller:spring name="pendulum_spring" plugin="libspring.so">
+				<alwaysOn> true </alwaysOn>
+				<updateRate> 10000 </updateRate>
+				<bodyName1> upright_link </bodyName1>
+				<bodyName2> pendulum_link </bodyName2>
+				<rotationalStiffness> ${spring_stiffness} </rotationalStiffness>
+			</controller:spring>
+		</gazebo>
+		<gazebo>
+			<controller:gazebo_ros_p3d name="p3d_base_controller" plugin="libgazebo_ros_p3d.so">
+						   <alwaysOn>true</alwaysOn>
+						   <updateRate>100.0</updateRate>
+						   <bodyName>pendulum_link</bodyName>
+						   <topicName>pendulum_pose_ground_truth</topicName>
+						   <gaussianNoise>0.01</gaussianNoise>
+						   <frameName>map</frameName>
+						   <xyzOffsets>25.7 25.7 0</xyzOffsets> <!-- initialize odometry for fake localization-->
+						   <rpyOffsets>0 0 0</rpyOffsets>
+						   <interface:position name="p3d_base_position"/>
+			</controller:gazebo_ros_p3d>
+		</gazebo>
 	</xacro:macro>
 </robot>
