Commit message: Starting to make planar model.  Currently broken.
git-svn-id: https://atrias.googlecode.com/svn/trunk@791 a504bc44-2baa-4cb8-4136-ba805e94d278

File: drl-sim/atrias/robots/simTest.urdf.xacro (robot description, xacro)
@@ -34,4 +34,59 @@
 	<xacro:macro name="atrias_robot">
 		<!--#########################################################################-->
+		<!--							Planar Motion								-->
+		<!--#########################################################################-->
+		<link name="world" />
+		<joint name="world_joint" type="fixed">
+			<origin xyz="0 0 0" rpy="0 0 0" />
+			<parent link="world" />
+			<child link="world_link"/>
+		</joint>
+		<link name="world_link">
+			<inertial>
+				<mass value="0.0000001"/>
+				<origin xyz="0 0 0" />
+				<inertia ixx="0.00000001" ixy="0" ixz="0"
+				         iyy="0.00000001" iyz="0"
+				         izz="0.00000001" />
+			</inertial>
+			<visual>
+				<origin xyz="0 0 0" rpy="0 0 0" />
+				<geometry>
+				  <cylinder length="${visual_motor_length}" radius="${visual_motor_radius}" />
+				</geometry>
+			</visual>
+			<collision>
+				<origin xyz="0 0 0" rpy="0 0 0" />
+				<geometry>
+					<cylinder length="${visual_motor_length}" radius="${visual_motor_radius}" />
+				</geometry>
+			</collision>
+		</link>
+		<gazebo reference="world_link">
+			<material>Gazebo/Blue</material>
+		</gazebo>
+		<joint name="planar_joint" type="prismatic">
+			<origin xyz="0 0 1.5" rpy="0 0 0" />
+			<axis xyz="0 0 1" />
+			<limit upper="100" lower="0" effort="1000000000" velocity="1000000000"/>
+			<parent link="world_link" />
+			<child link="planar_link"/>
+		</joint>
+		<link name="planar_link">
+			<inertial>
+				<mass value="0.0000001"/>
+				<origin xyz="0 0 0" />
+				<inertia ixx="0.00000001" ixy="0" ixz="0"
+				         iyy="0.00000001" iyz="0"
+				         izz="0.00000001" />
+			</inertial>
+		</link>
+		<joint name="body_no_twist_joint" type="continuous">
+			<origin xyz="0 0 0" rpy="0 0 0" />
+			<axis xyz="0 1 0" />
+			<parent link="planar_link" />
+			<child link="body_link"/>
+		</joint>
+		<!--#########################################################################-->
 		<!--								Body                                     -->
 		<!--#########################################################################-->
@@ -39,5 +94,5 @@
 			<inertial>
 				<mass value="${body_mass}" />
-				<origin xyz="0 0 0" />
+				<origin xyz="0 0.5 0" />
 			<inertia ixx="0.8" ixy="0.01" ixz="0.01"
 					 iyy="0.7" iyz="0.01"

Commit message: Planar constraint working
git-svn-id: https://atrias.googlecode.com/svn/trunk@792 a504bc44-2baa-4cb8-4136-ba805e94d278

File: drl-sim/atrias/robots/simTest.urdf.xacro (robot description, xacro)
@@ -37,6 +37,7 @@
 		<!--#########################################################################-->
 		<link name="world" />
-		<joint name="world_joint" type="fixed">
-			<origin xyz="0 0 0" rpy="0 0 0" />
+		<joint name="world_joint" type="continuous">
+			<origin xyz="0 0 0" rpy="0 0 0" />
+			<axis xyz="0 1 0" />
 			<parent link="world" />
 			<child link="world_link"/>
@@ -44,40 +45,25 @@
 		<link name="world_link">
 			<inertial>
-				<mass value="0.0000001"/>
-				<origin xyz="0 0 0" />
-				<inertia ixx="0.00000001" ixy="0" ixz="0"
-				         iyy="0.00000001" iyz="0"
-				         izz="0.00000001" />
-			</inertial>
-			<visual>
-				<origin xyz="0 0 0" rpy="0 0 0" />
-				<geometry>
-				  <cylinder length="${visual_motor_length}" radius="${visual_motor_radius}" />
-				</geometry>
-			</visual>
-			<collision>
-				<origin xyz="0 0 0" rpy="0 0 0" />
-				<geometry>
-					<cylinder length="${visual_motor_length}" radius="${visual_motor_radius}" />
-				</geometry>
-			</collision>
-		</link>
-		<gazebo reference="world_link">
-			<material>Gazebo/Blue</material>
-		</gazebo>
+				<mass value="0.00001"/>
+				<origin xyz="0 0 0" />
+				<inertia ixx="0.00001" ixy="0" ixz="0"
+				         iyy="0.00001" iyz="0"
+				         izz="0.00001" />
+			</inertial>
+		</link>
 		<joint name="planar_joint" type="prismatic">
 			<origin xyz="0 0 1.5" rpy="0 0 0" />
 			<axis xyz="0 0 1" />
-			<limit upper="100" lower="0" effort="1000000000" velocity="1000000000"/>
+			<limit upper="100" lower="-100" effort="1000000000" velocity="1000000000"/>
 			<parent link="world_link" />
-			<child link="planar_link"/>
-		</joint>
-		<link name="planar_link">
-			<inertial>
-				<mass value="0.0000001"/>
-				<origin xyz="0 0 0" />
-				<inertia ixx="0.00000001" ixy="0" ixz="0"
-				         iyy="0.00000001" iyz="0"
-				         izz="0.00000001" />
+			<child link="body_no_twist_link"/>
+		</joint>
+		<link name="body_no_twist_link">
+			<inertial>
+				<mass value="0.00001"/>
+				<origin xyz="0 0 0" />
+				<inertia ixx="0.00001" ixy="0" ixz="0"
+				         iyy="0.00001" iyz="0"
+				         izz="0.00001" />
 			</inertial>
 		</link>
@@ -85,5 +71,5 @@
 			<origin xyz="0 0 0" rpy="0 0 0" />
 			<axis xyz="0 1 0" />
-			<parent link="planar_link" />
+			<parent link="body_no_twist_link" />
 			<child link="body_link"/>
 		</joint>

Commit message: Correct inertias for Atrias 2.0
git-svn-id: https://atrias.googlecode.com/svn/trunk@793 a504bc44-2baa-4cb8-4136-ba805e94d278

File: drl-sim/atrias/robots/simTest.urdf.xacro (robot description, xacro)
@@ -23,8 +23,9 @@
 	<property name="body_mass" value="0.500" />
 	<property name="motor_mass" value="0.500" />
-	<property name="thigh_mass" value="0.500" />
-	<property name="shin_mass" value="0.350" />
-	<property name="lower_mass" value="0.350" />
-	<property name="fourBar_mass" value="0.500" />
+	<property name="thigh_mass" value="3.132" />
+	<property name="shin_mass" value="3.137" />
+	<property name="lower_mass" value="0.204" />
+	<property name="fourBar_mass" value="0.166" />
+	<property name="toe_mass" value="0.087" />
 	<property name="spring_stiffness" value="10000" />
 	<property name="motor_damping" value="10000000" />
@@ -79,9 +80,9 @@
 		<link name="body_link">
 			<inertial>
+				<origin xyz="0 0 0.002" />
 				<mass value="${body_mass}" />
-				<origin xyz="0 0.5 0" />
-			<inertia ixx="0.8" ixy="0.01" ixz="0.01"
-					 iyy="0.7" iyz="0.01"
-				     izz="0.9" />
+				<inertia ixx="0.0932" ixy="0.0044" ixz="-0.0019"
+						 iyy="0.0833" iyz="-0.0102"
+					     izz="0.0785" />
 			</inertial>
 			<visual>
@@ -115,8 +116,8 @@
 			<inertial>
 				<mass value="${motor_mass}"/>
-				<origin xyz="0 0 0" />
-				<inertia ixx="5" ixy="0" ixz="0"
-				         iyy="5" iyz="0"
-				         izz="5" />
+				<origin xyz="0 -0.044 0" />
+				<inertia ixx="4" ixy="0" ixz="0"
+				         iyy="7.25" iyz="0"
+				         izz="4" />
 			</inertial>
 			<visual>
@@ -159,8 +160,8 @@
 			<inertial>
 				<mass value="${motor_mass}"/>
-				<origin xyz="0 0 0" />
-				<inertia ixx="5" ixy="0" ixz="0"
-				         iyy="5" iyz="0"
-				         izz="5" />
+				<origin xyz="0 0.044 0" />
+				<inertia ixx="4" ixy="0" ixz="0"
+				         iyy="7.25" iyz="0"
+				         izz="4" />
 			</inertial>
 			<visual>
@@ -203,8 +204,8 @@
 			<inertial>
 				<mass value="${thigh_mass}"/>
-				<origin xyz="${thigh_length/SQRT_2/2} 0 ${-thigh_length/SQRT_2/2}" />
-				<inertia ixx="0.01910" ixy="0" ixz="0"
-				         iyy="0.01910" iyz="0"
-				         izz="0.01910" />
+				<origin xyz="0.100 -0.020 -0.011" />
+				<inertia ixx="0.0339" ixy="0.0056" ixz="-0.0179"
+				         iyy="0.0688" iyz="-0.0017"
+				         izz="0.0512" />
 			</inertial>
 			<visual>
@@ -238,8 +239,8 @@
 			<inertial>
 				<mass value="${shin_mass}"/>
-				<origin xyz="${-shin_length/SQRT_2/2} 0 ${-shin_length/SQRT_2/2}" />
-				<inertia ixx="0.02116" ixy="0" ixz="0"
-				         iyy="0.02116" iyz="0"
-				         izz="0.02116" />
+				<origin xyz="-0.0979 0.0200 -0.0081" />
+				<inertia ixx="0.0309" ixy="0.0054" ixz="0.0154"
+				         iyy="0.0637" iyz="0.0014"
+				         izz="0.0493" />
 			</inertial>
 			<visual>
@@ -273,8 +274,8 @@
 			<inertial>
 				<mass value="${lower_mass}"/>
-				<origin xyz="${-lower_length/SQRT_2/2} 0 ${-lower_length/SQRT_2/2}" />
-				<inertia ixx="0.00633" ixy="0" ixz="0"
-				         iyy="0.00633" iyz="0"
-				         izz="0.00633" />
+				<origin xyz="-0.127 0 -0.141" />
+				<inertia ixx="0.0027" ixy="0" ixz="0.0026"
+				         iyy="0.0054" iyz="0"
+				         izz="0.0028" />
 			</inertial>
 			<visual>
@@ -308,8 +309,8 @@
 			<inertial>
 				<mass value="${fourBar_mass}"/>
-				<origin xyz="${fourBar_length/SQRT_2/2} 0 ${-fourBar_length/SQRT_2/2}" />
-				<inertia ixx="0.006243" ixy="0" ixz="0"
-				         iyy="0.0061243" iyz="0"
-				         izz="0.0001243" />
+				<origin xyz="0.1633 0 -0.1633" />
+				<inertia ixx="0.0033" ixy="0" ixz="-0.0032"
+				         iyy="0.0063" iyz="0"
+				         izz="0.0033" />
 			</inertial>
 			<visual>
@@ -351,5 +352,5 @@
 		<link name="toe_link">
 			<inertial>
-				<mass value="0.000001"/>
+				<mass value="${toe_mass}"/>
 				<origin xyz="0 0 0" />
 				<inertia ixx="0.0000001" ixy="0" ixz="0"
