Commit message: Correct boom inertias
git-svn-id: https://atrias.googlecode.com/svn/trunk@840 a504bc44-2baa-4cb8-4136-ba805e94d278

File: drl-sim/atrias_sim/robots/atrias20_boom_header.urdf.xacro (robot description, xacro)
@@ -18,8 +18,8 @@
 	<include filename="boom21.urdf.xacro" />
 	<!-- constrains and builds the atrias leg model.
-		NOTE: initial_pitch_angle must be less than 25 Deg -->
-	<xacro:boom21 initial_pitch_angle="${M_PI/180*15}" child_link="leg_hip_link" />
+		NOTE: initial_pitch_angle must be inside +-25 Deg -->
+	<xacro:boom21 initial_pitch_angle="${M_PI/180*15}" child_link="leg_hip_link" child_offset="0.075"/>
 	<xacro:atrias_leg hip_link="leg_hip_link">
-		<origin xyz="0 0 0.002" />
+		<origin xyz="0 0 0.002" />	<!-- Center of rotation to center of mass   -->
 	</xacro:atrias_leg>
 	<!-- initializes the all-in-one controller with the correct link names, etc. -->

File: drl-sim/atrias_sim/robots/atrias20_leg.urdf.xacro (robot description, xacro)
@@ -35,7 +35,7 @@
 	<property name="toe_mass" value="0.087" />
 	<!-- Spring/Damping Coefficients -->
-	<property name="spring_stiffness" value="10000" />
-	<property name="motor_damping" value="10000000" />
-	<property name="motor_friction" value="10000000" />
+	<property name="spring_stiffness" value="1200" />			<!-- N*m/rad -->
+	<property name="motor_damping" value="${2*0.5*34.64}" />	<!-- 2*Zeta*sqrt(K) (Guessed Zeta)-->
+	<property name="motor_friction" value="10" />				<!-- Guess -->
 	<property name="leg_damping" value="0" />
 	<property name="leg_friction" value="0" />
@@ -77,5 +77,5 @@
 			<parent link="${hip_link}" />
 			<child link="thighMotor_link" />
-			<limit lower="${-M_PI/4-0.3054}" upper="${-M_PI/4+2.3562}" effort="10000000000000" velocity="100000000000000" />
+			<limit lower="${-M_PI/4-0.3054}" upper="${-M_PI/4+2.3562}" effort="1000000" velocity="1000000" />
 			<dynamics damping="${motor_damping}" friction="${motor_friction}" />
 		</joint>
@@ -314,4 +314,5 @@
 		<joint name="lower_toe_joint" type="continuous">
 			<axis xyz="1 0 0" />
+			<origin xyz="${-fourBar_length/SQRT_2} 0 ${-fourBar_length/SQRT_2}" rpy="0 0 0" />
 			<parent link="lower_link" />
 			<child link="toe_link"/>

File: drl-sim/atrias_sim/robots/boom21.urdf.xacro (robot description, xacro)
@@ -23,5 +23,5 @@
 	<property name="yaw_radius" value="0.02" />
 	<property name="pitch_radius" value="0.02" />
-	<xacro:macro name="boom21" params="initial_pitch_angle child_link">
+	<xacro:macro name="boom21" params="initial_pitch_angle child_link child_offset">
 		<link name="world" />
 		<!--#########################################################################-->
@@ -29,6 +29,6 @@
 		<!--#########################################################################-->
 		<joint name="upright_yaw_joint" type="continuous">
-			<axis xyz="0 0 1" />
-			<origin xyz="0 0 ${upright_length}" rpy="0 0 0" />
+			<axis xyz="0 1 0" />
+			<origin xyz="0 0 ${upright_length}" rpy="${M_PI/2} 0 0" />	<!-- x along boom, y upwards -->
 			<parent link="world" />
 			<child link="yaw_link"/>
@@ -37,11 +37,11 @@
 			<inertial>
 				<mass value="${yaw_mass}"/>
-				<origin xyz="0 ${yaw_length/3} 0" rpy="0 0 0" />
-				<inertia ixx="0.01" ixy="0" ixz="0"
-				         iyy="0.01" iyz="0"
-				         izz="0.01" />
+				<origin xyz="0.15069 0.0007 -0.00561" />
+				<inertia ixx="3.7013" ixy="2.3205" ixz="0.0103"
+				         iyy="2.7884" iyz="0.0229"
+				         izz="6.2744" />
 			</inertial>
-	<!--		<visual>
-				<origin xyz="0 ${yaw_length/SQRT_2/2} ${yaw_length/SQRT_2/2}" rpy="${-M_PI/4} 0 0" />
+		<visual>
+				<origin xyz="${yaw_length/SQRT_2/2} ${yaw_length/SQRT_2/2} 0" rpy="0 ${M_PI/2} ${M_PI/4}" />
 				<geometry>
 				  <cylinder length="${yaw_length}" radius="${yaw_radius}" />
@@ -49,10 +49,10 @@
 			</visual>
 			<collision>
-				<origin xyz="0 ${yaw_length/SQRT_2/2} ${yaw_length/SQRT_2/2}" rpy="${-M_PI/4} 0 0" />
+				<origin xyz="${yaw_length/SQRT_2/2} ${yaw_length/SQRT_2/2} 0" rpy="0 ${M_PI/2} ${M_PI/4}" />
 				<geometry>
 					<cylinder length="${yaw_length}" radius="${yaw_radius}" />
 				</geometry>
 			</collision>
--->		</link>
+		</link>
 		<gazebo reference="yaw_link">
 			<material>Gazebo/Red</material>
@@ -62,6 +62,6 @@
 		<!--#########################################################################-->
 		<joint name="yaw_pitch_joint" type="continuous">
-			<axis xyz="1 0 0" />
-			<origin xyz="0 0 0" rpy="${initial_pitch_angle} 0 0" />
+			<axis xyz="0 0 1" />
+			<origin xyz="0 0 0" rpy="0 0 ${initial_pitch_angle}" />
 			<limit lower="${-M_PI/180*25}" upper="${M_PI/180*25}" effort="100000" velocity="100000" />
 			<parent link="yaw_link" />
@@ -71,11 +71,11 @@
 			<inertial>
 				<mass value="${pitch_mass}"/>
-				<origin xyz="0 ${pitch_length/2} 0" />
-				<inertia ixx="0.01" ixy="0" ixz="0"
-				         iyy="0.01" iyz="0"
-				         izz="0.01" />
+				<origin xyz="1.09153 0.00637 0.0" />
+				<inertia ixx="0.0069" ixy="0.0111" ixz="0.0"
+				         iyy="0.9699" iyz="0.0"
+				         izz="0.9712" />
 			</inertial>
-	<!--		<visual>
-				<origin xyz="0 ${pitch_length/2} 0" rpy="${M_PI/2} 0 0" />
+		<visual>
+				<origin xyz="${pitch_length/2} 0 0" rpy="0 ${M_PI/2} 0" />
 				<geometry>
 				  <cylinder length="${pitch_length}" radius="${pitch_radius}" />
@@ -83,10 +83,10 @@
 			</visual>
 			<collision>
-				<origin xyz="0 ${pitch_length/2} 0" rpy="${M_PI/2} 0 0" />
+				<origin xyz="${pitch_length/2} 0 0" rpy="0 ${M_PI/2} 0" />
 				<geometry>
 					<cylinder length="${pitch_length}" radius="${pitch_radius}" />
 				</geometry>
 			</collision>
--->		</link>
+		</link>
 		<gazebo reference="pitch_link">
 			<material>Gazebo/Red</material>
@@ -97,5 +97,5 @@
 		<joint name="pitch_roll_joint" type="continuous">
 			<axis xyz="0 1 0" />
-			<origin xyz="0 ${pitch_length} 0" rpy="0 0 0" />
+			<origin xyz="${pitch_length + child_offset} 0 0" rpy="0 ${-M_PI/2} ${-M_PI/2}" /> <!-- y along boom, z upwards -->
 			<parent link="pitch_link" />
 			<child link="${child_link}"/>

Commit message: Planar and Boom models completely defined and functional
git-svn-id: https://atrias.googlecode.com/svn/trunk@869 a504bc44-2baa-4cb8-4136-ba805e94d278

File: drl-sim/atrias_sim/robots/atrias20_boom_header.urdf.xacro (robot description, xacro)
@@ -14,4 +14,9 @@
 	<!-- Constants -->
 	<property name="M_PI" value="3.14159"/>
+	<property name="angle" value="${M_PI/180*1}" />
+    <!-- Note: "a" is the calculated value of angle because of xacro limitations -->
+	<property name="a" value="0.01745" />
+	<property name="cos_a" value="${1 - a*a/2 + a*a*a*a/4/3/2 - a*a*a*a*a*a/6/5/4/3/2}" />
+	<property name="sin_a" value="${a - a*a*a/3/2 + a*a*a*a*a/5/4/3/2 - a*a*a*a*a*a*a/7/6/5/4/3/2}" />
 	<!-- get robot model macro -->
 	<include filename="atrias20_leg.urdf.xacro" />
@@ -19,7 +24,8 @@
 	<!-- constrains and builds the atrias leg model.
 		NOTE: initial_pitch_angle must be inside +-25 Deg -->
-	<xacro:boom21 initial_pitch_angle="${M_PI/180*15}" child_link="leg_hip_link" child_offset="0.075"/>
-	<xacro:atrias_leg hip_link="leg_hip_link">
+	<xacro:boom21 initial_pitch_angle="${angle}" child_link="leg_hip_link" child_offset="0.075"/>
+	<xacro:atrias_leg hip_link="leg_hip_link" >
 		<origin xyz="0 0 0.002" />	<!-- Center of rotation to center of mass   -->
+		<axis>${cos_a} 0 ${sin_a}</axis>  <!-- Axis of rotation for 4-bar linkage -->
 	</xacro:atrias_leg>
 	<!-- initializes the all-in-one controller with the correct link names, etc. -->

File: drl-sim/atrias_sim/robots/atrias20_leg.urdf.xacro (robot description, xacro)
@@ -41,5 +41,5 @@
 	<property name="leg_friction" value="0" />
 	<!-- macro to use in the header file when parsed by xacro -->
-	<xacro:macro name="atrias_leg" params="hip_link *origin">
+	<xacro:macro name="atrias_leg" params="hip_link *origin *axis" >
 		<!--#########################################################################-->
 		<!--								Body                                     -->
@@ -300,4 +300,5 @@
 		<!--							Four Bar Linkage Joint						-->
 		<!--#########################################################################-->
+		<!-- Calculate four bar linkage axis -->
 		<gazebo>
 			<joint:hinge name="lower_fourBar_joint">
@@ -305,5 +306,5 @@
 				<body2>fourBar_link</body2>
 				<anchor>lower_link</anchor>
-				<axis>0 1 0</axis>
+				<insert_block name="axis" />
 				<anchorOffset>${-(lower_length-0.15)/SQRT_2} 0 ${-(lower_length-0.15)/SQRT_2}</anchorOffset>
 			</joint:hinge>

File: drl-sim/atrias_sim/robots/atrias20_planar_header.urdf.xacro (robot description, xacro)
@@ -19,4 +19,5 @@
 	<xacro:atrias_leg hip_link="leg_hip_link">
 		<origin xyz="0 0 0.002" />
+		<axis>0 1 0</axis>  <!-- Axis of rotation for 4-bar linkage -->
 	</xacro:atrias_leg>
 	<!-- initializes the all-in-one controller with the correct link names, etc. -->

File: drl-sim/atrias_sim/robots/boom21.urdf.xacro (robot description, xacro)
@@ -14,13 +14,12 @@
 	<property name="SQRT_2" value="1.41421356"/>
 	<!-- Physical Properties -->
-	<property name="upright_length" value="0.5" />
-	<property name="yaw_length" value="2" />
+	<property name="upright_length" value="0.93" />
+	<property name="yaw_length" value="2.4" />
 	<property name="pitch_length" value="1.795" />
 	<property name="yaw_mass" value="14.19014" />
 	<property name="pitch_mass" value="2.66782" />
 	<!-- Visual Properties -->
-	<property name="upright_radius" value="0.02" />
-	<property name="yaw_radius" value="0.02" />
-	<property name="pitch_radius" value="0.02" />
+	<property name="yaw_radius" value="0.034" />
+	<property name="pitch_radius" value="0.049" />
 	<xacro:macro name="boom21" params="initial_pitch_angle child_link child_offset">
 		<link name="world" />
@@ -43,5 +42,5 @@
 			</inertial>
 		<visual>
-				<origin xyz="${yaw_length/SQRT_2/2} ${yaw_length/SQRT_2/2} 0" rpy="0 ${M_PI/2} ${M_PI/4}" />
+				<origin xyz="1 0.7 0" rpy="0 ${M_PI/2} 0.6107" />
 				<geometry>
 				  <cylinder length="${yaw_length}" radius="${yaw_radius}" />
@@ -49,5 +48,5 @@
 			</visual>
 			<collision>
-				<origin xyz="${yaw_length/SQRT_2/2} ${yaw_length/SQRT_2/2} 0" rpy="0 ${M_PI/2} ${M_PI/4}" />
+				<origin xyz="1 0.7 0" rpy="0 ${M_PI/2} 0.6107" />
 				<geometry>
 					<cylinder length="${yaw_length}" radius="${yaw_radius}" />
