Commit message: Added and completed biped template.  Working.
git-svn-id: https://atrias.googlecode.com/svn/trunk@884 a504bc44-2baa-4cb8-4136-ba805e94d278

File: drl-sim/atrias_sim/robots/atrias20_boom_header.urdf.xacro (robot description, xacro)
@@ -24,6 +24,6 @@
 	<!-- constrains and builds the atrias leg model.
 		NOTE: initial_pitch_angle must be inside +-25 Deg -->
-	<xacro:boom21 initial_pitch_angle="${angle}" child_link="leg_hip_link" child_offset="0.075"/>
-	<xacro:atrias_leg hip_link="leg_hip_link" >
+	<xacro:boom21 initial_pitch_angle="${angle}" child_link="leg_hip_link1" child_offset="0.075" child_pitch="0" biped="0" />
+	<xacro:atrias_leg hip_link="leg_hip_link" suffix="1" >
 		<origin xyz="0 0 0.002" />	<!-- Center of rotation to center of mass   -->
 		<axis>${cos_a} 0 ${sin_a}</axis>  <!-- Axis of rotation for 4-bar linkage -->
@@ -34,9 +34,9 @@
 			<alwaysOn> true </alwaysOn>
 			<updateRate> 1000 </updateRate>
-			<bodyName> leg_hip_link </bodyName>
-			<motorAName> thighMotor_link </motorAName>
-			<motorBName> shinMotor_link </motorBName>
-			<legAName> thigh_link </legAName>
-			<legBName> shin_link </legBName>
+			<bodyName> leg_hip_link1 </bodyName>
+			<motorAName> thighMotor_link1 </motorAName>
+			<motorBName> shinMotor_link1 </motorBName>
+			<legAName> thigh_link1 </legAName>
+			<legBName> shin_link1 </legBName>
 		</controller:all_in_one_controller_wrapper>
 	</gazebo>

File: drl-sim/atrias_sim/robots/atrias20_leg.urdf.xacro (robot description, xacro)
@@ -27,6 +27,6 @@
 	<property name="fourBar_length" value="0.500" />
 	<!-- Link Masses -->
-	<property name="body_mass" value="0.500" />
-	<property name="motor_mass" value="0.500" />
+	<property name="body_mass" value="11.61" />
+	<property name="motor_mass" value="1.273" />
 	<property name="thigh_mass" value="3.132" />
 	<property name="shin_mass" value="3.137" />
@@ -41,9 +41,9 @@
 	<property name="leg_friction" value="0" />
 	<!-- macro to use in the header file when parsed by xacro -->
-	<xacro:macro name="atrias_leg" params="hip_link *origin *axis" >
+	<xacro:macro name="atrias_leg" params="hip_link suffix *origin *axis" >
 		<!--#########################################################################-->
 		<!--								Body                                     -->
 		<!--#########################################################################-->
-		<link name="${hip_link}">
+		<link name="${hip_link}${suffix}">
 			<inertial>
 				<insert_block name="origin" />
@@ -66,5 +66,5 @@
 			</collision>
 		</link>
-		<gazebo reference="${hip_link}">
+		<gazebo reference="${hip_link}${suffix}">
 			<material>Gazebo/BumpyMetal</material>
 		</gazebo>
@@ -72,13 +72,13 @@
 		<!--								Thigh Motor                              -->
 		<!--#########################################################################-->
-		<joint name="hip_thighMotor_joint" type="revolute">
+		<joint name="hip_thighMotor_joint${suffix}" type="revolute">
 			<axis xyz="0 1 0" />
 			<origin xyz="0 0 0" rpy="0 0 0" />
-			<parent link="${hip_link}" />
-			<child link="thighMotor_link" />
+			<parent link="${hip_link}${suffix}" />
+			<child link="thighMotor_link${suffix}" />
 			<limit lower="${-M_PI/4-0.3054}" upper="${-M_PI/4+2.3562}" effort="1000000" velocity="1000000" />
 			<dynamics damping="${motor_damping}" friction="${motor_friction}" />
 		</joint>
-		<link name="thighMotor_link">
+		<link name="thighMotor_link${suffix}">
 			<inertial>
 				<mass value="${motor_mass}"/>
@@ -101,13 +101,13 @@
 			</collision>
 		</link>
-		<gazebo reference="thighMotor_link">
+		<gazebo reference="thighMotor_link${suffix}">
 			<material> Gazebo/Green </material>
 		</gazebo>
 		<gazebo>
-			<controller:spring name="thighSpring" plugin="libspring.so">
+			<controller:spring name="thighSpring${suffix}" plugin="libspring.so">
 				<alwaysOn> true </alwaysOn>
 				<updateRate> 10000 </updateRate>
-				<bodyName1> thighMotor_link </bodyName1>
-				<bodyName2> thigh_link </bodyName2>
+				<bodyName1> thighMotor_link${suffix} </bodyName1>
+				<bodyName2> thigh_link${suffix} </bodyName2>
 				<rotationalStiffness> ${spring_stiffness} </rotationalStiffness>
 			</controller:spring>
@@ -116,13 +116,13 @@
 		<!--					Shin Motor                                           -->
 		<!--#########################################################################-->
-		<joint name="hip_shinMotor_joint" type="revolute">
+		<joint name="hip_shinMotor_joint${suffix}" type="revolute">
 			<axis xyz="0 1 0" />
 			<origin xyz="0 0 0" rpy="0 0 0" />
-			<parent link="${hip_link}" />
-			<child link="shinMotor_link"/>
+			<parent link="${hip_link}${suffix}" />
+			<child link="shinMotor_link${suffix}"/>
 			<limit lower="${-5*M_PI/4+2.8362}" upper="${-5*M_PI/4+5.4978}" effort="10000000000000" velocity="100000000000000" />
 			<dynamics damping="${motor_damping}" friction="${motor_friction}" />
 		</joint>
-		<link name="shinMotor_link">
+		<link name="shinMotor_link${suffix}">
 			<inertial>
 				<mass value="${motor_mass}"/>
@@ -145,13 +145,13 @@
 			</collision>
 		</link>
-		<gazebo reference="shinMotor_link">
+		<gazebo reference="shinMotor_link${suffix}">
 			<material>Gazebo/Green</material>
 		</gazebo>
 		<gazebo>
-			<controller:spring name="shinSpring" plugin="libspring.so">
+			<controller:spring name="shinSpring${suffix}" plugin="libspring.so">
 				<alwaysOn> true </alwaysOn>
 				<updateRate> 10000 </updateRate>
-				<bodyName1> shinMotor_link </bodyName1>
-				<bodyName2> shin_link </bodyName2>
+				<bodyName1> shinMotor_link${suffix} </bodyName1>
+				<bodyName2> shin_link${suffix} </bodyName2>
 				<rotationalStiffness> ${spring_stiffness} </rotationalStiffness>
 			</controller:spring>
@@ -160,13 +160,13 @@
 		<!--							 Thigh 										-->
 		<!--#########################################################################-->
-		<joint name="body_thigh_joint" type="continuous">
+		<joint name="body_thigh_joint${suffix}" type="continuous">
 			<axis xyz="0 1 0" />
 			<origin xyz="0 0 0" rpy="0 0 0" />
-			<parent link="${hip_link}" />
-			<child link="thigh_link"/>
+			<parent link="${hip_link}${suffix}" />
+			<child link="thigh_link${suffix}"/>
 			<!--limit lower="${-M_PI/4-0.6545}" upper="${-M_PI/4+2.7053}" effort="1000000000000" velocity="100000000000000" /-->
 			<dynamics damping="${leg_damping}" friction="${leg_friction}" />
 		</joint>
-		<link name="thigh_link">
+		<link name="thigh_link${suffix}">
 			<inertial>
 				<mass value="${thigh_mass}"/>
@@ -189,5 +189,5 @@
 			</collision>
 		</link>
-		<gazebo reference="thigh_link">
+		<gazebo reference="thigh_link${suffix}">
 			<material>Gazebo/Red</material>
 		</gazebo>
@@ -195,13 +195,13 @@
 		<!--							 Shin 			 							-->
 		<!--#########################################################################-->
-		<joint name="body_shin_joint" type="continuous">
+		<joint name="body_shin_joint${suffix}" type="continuous">
 			<axis xyz="0 1 0" />
 			<origin xyz="0 0 0" rpy="0 0 0" />
-			<parent link="${hip_link}" />
-			<child link="shin_link"/>
+			<parent link="${hip_link}${suffix}" />
+			<child link="shin_link${suffix}"/>
 			<!--limit lower="${-5*M_PI/4+2.4871}" upper="${-5*M_PI/4+5.4978}" effort="100000000000" velocity="100000000000000" /-->
 			<dynamics damping="${leg_damping}" friction="${leg_friction}" />
 		</joint>
-		<link name="shin_link">
+		<link name="shin_link${suffix}">
 			<inertial>
 				<mass value="${shin_mass}"/>
@@ -224,5 +224,5 @@
 			</collision>
 		</link>
-		<gazebo reference="shin_link">
+		<gazebo reference="shin_link${suffix}">
 			<material>Gazebo/Red</material>
 		</gazebo>
@@ -230,13 +230,13 @@
 		<!--								 Lower Link					 			-->
 		<!--#########################################################################-->
-		<joint name="thigh_lower_joint" type="continuous">
+		<joint name="thigh_lower_joint${suffix}" type="continuous">
 			<axis xyz="0 1 0" />
 			<origin xyz="${thigh_length/SQRT_2} 0 ${-thigh_length/SQRT_2}" rpy="0 0 0" />
-			<parent link="thigh_link" />
-			<child link="lower_link"/>
+			<parent link="thigh_link${suffix}" />
+			<child link="lower_link${suffix}"/>
 			<limit lower="${-M_PI/2}" upper="${M_PI/2}" effort="10000000000000" velocity="100000000000000" />
 			<dynamics damping="${leg_damping}" friction="${leg_friction}" />
 		</joint>
-		<link name="lower_link">
+		<link name="lower_link${suffix}">
 			<inertial>
 				<mass value="${lower_mass}"/>
@@ -259,5 +259,5 @@
 			</collision>
 		</link>
-		<gazebo reference="lower_link">
+		<gazebo reference="lower_link${suffix}">
 			<material>Gazebo/Red</material>
 		</gazebo>
@@ -265,13 +265,13 @@
 		<!--								 Four Bar	 							-->
 		<!--#########################################################################-->
-		<joint name="shin_fourBar_joint" type="continuous">
+		<joint name="shin_fourBar_joint${suffix}" type="continuous">
 			<axis xyz="0 1 0" />
 			<origin xyz="${-shin_length/SQRT_2} 0 ${-shin_length/SQRT_2}" rpy="0 0 0" />
-			<parent link="shin_link" />
-			<child link="fourBar_link"/>
+			<parent link="shin_link${suffix}" />
+			<child link="fourBar_link${suffix}"/>
 			<limit lower="${-M_PI/2}" upper="${M_PI/2}" effort="10000000000000" velocity="100000000000000" />
 			<dynamics damping="${leg_damping}" friction="${leg_friction}" />
 		</joint>
-		<link name="fourBar_link">
+		<link name="fourBar_link${suffix}">
 			<inertial>
 				<mass value="${fourBar_mass}"/>
@@ -294,5 +294,5 @@
 			</collision>
 		</link>
-		<gazebo reference="fourBar_link">
+		<gazebo reference="fourBar_link${suffix}">
 			<material>Gazebo/Red</material>
 		</gazebo>
@@ -300,10 +300,9 @@
 		<!--							Four Bar Linkage Joint						-->
 		<!--#########################################################################-->
-		<!-- Calculate four bar linkage axis -->
 		<gazebo>
-			<joint:hinge name="lower_fourBar_joint">
-				<body1>lower_link</body1>
-				<body2>fourBar_link</body2>
-				<anchor>lower_link</anchor>
+			<joint:hinge name="lower_fourBar_joint${suffix}">
+				<body1>lower_link${suffix}</body1>
+				<body2>fourBar_link${suffix}</body2>
+				<anchor>lower_link${suffix}</anchor>
 				<insert_block name="axis" />
 				<anchorOffset>${-(lower_length-0.15)/SQRT_2} 0 ${-(lower_length-0.15)/SQRT_2}</anchorOffset>
@@ -313,11 +312,11 @@
 		<!--							Toe											-->
 		<!--#########################################################################-->
-		<joint name="lower_toe_joint" type="continuous">
+		<joint name="lower_toe_joint${suffix}" type="continuous">
 			<axis xyz="1 0 0" />
 			<origin xyz="${-fourBar_length/SQRT_2} 0 ${-fourBar_length/SQRT_2}" rpy="0 0 0" />
-			<parent link="lower_link" />
-			<child link="toe_link"/>
-		</joint>
-		<link name="toe_link">
+			<parent link="lower_link${suffix}" />
+			<child link="toe_link${suffix}"/>
+		</joint>
+		<link name="toe_link${suffix}">
 			<inertial>
 				<mass value="${toe_mass}"/>
@@ -340,5 +339,5 @@
 			</collision>
 		</link>
-		<gazebo reference="toe_link">
+		<gazebo reference="toe_link${suffix}">
 			<material>Gazebo/Red</material>
 		</gazebo>

File: drl-sim/atrias_sim/robots/atrias20_planar_header.urdf.xacro (robot description, xacro)
@@ -16,6 +16,6 @@
 	<include filename="planar_constraint.urdf.xacro" />
 	<!-- constrains and builds the atrias leg model -->
-	<xacro:planar_constraint child_attachment_link="leg_hip_link" />
-	<xacro:atrias_leg hip_link="leg_hip_link">
+	<xacro:planar_constraint child_attachment_link="leg_hip_link1" />
+	<xacro:atrias_leg hip_link="leg_hip_link" suffix="1" >
 		<origin xyz="0 0 0.002" />
 		<axis>0 1 0</axis>  <!-- Axis of rotation for 4-bar linkage -->
@@ -26,9 +26,9 @@
 			<alwaysOn> true </alwaysOn>
 			<updateRate> 1000 </updateRate>
-			<bodyName> leg_hip_link </bodyName>
-			<motorAName> thighMotor_link </motorAName>
-			<motorBName> shinMotor_link </motorBName>
-			<legAName> thigh_link </legAName>
-			<legBName> shin_link </legBName>
+			<bodyName> leg_hip_link1 </bodyName>
+			<motorAName> thighMotor_link1 </motorAName>
+			<motorBName> shinMotor_link1 </motorBName>
+			<legAName> thigh_link1 </legAName>
+			<legBName> shin_link1 </legBName>
 		</controller:all_in_one_controller_wrapper>
 	</gazebo>

File: drl-sim/atrias_sim/robots/boom21.urdf.xacro (robot description, xacro)
@@ -22,5 +22,5 @@
 	<property name="yaw_radius" value="0.034" />
 	<property name="pitch_radius" value="0.049" />
-	<xacro:macro name="boom21" params="initial_pitch_angle child_link child_offset">
+	<xacro:macro name="boom21" params="initial_pitch_angle child_link child_offset child_pitch biped">
 		<link name="world" />
 		<!--#########################################################################-->
@@ -96,5 +96,5 @@
 		<joint name="pitch_roll_joint" type="continuous">
 			<axis xyz="0 1 0" />
-			<origin xyz="${pitch_length + child_offset} 0 0" rpy="0 ${-M_PI/2} ${-M_PI/2}" /> <!-- y along boom, z upwards -->
+			<origin xyz="${pitch_length + child_offset} ${-0.08*biped} 0" rpy="${-M_PI/2*biped} ${-M_PI/2 + M_PI/2*biped} ${-M_PI/2 + M_PI/2*biped + child_pitch}" />
 			<parent link="pitch_link" />
 			<child link="${child_link}"/>
