Commit message: Corrected last boom joint for biped
git-svn-id: https://atrias.googlecode.com/svn/trunk@896 a504bc44-2baa-4cb8-4136-ba805e94d278

File: drl-sim/atrias_sim/robots/boom21.urdf.xacro (robot description, xacro)
@@ -28,6 +28,6 @@
 		<!--#########################################################################-->
 		<joint name="upright_yaw_joint" type="continuous">
+			<origin xyz="0 0 ${upright_length}" rpy="${M_PI/2} 0 0" />	<!-- x along boom, y upwards -->
 			<axis xyz="0 1 0" />
-			<origin xyz="0 0 ${upright_length}" rpy="${M_PI/2} 0 0" />	<!-- x along boom, y upwards -->
 			<parent link="world" />
 			<child link="yaw_link"/>
@@ -61,6 +61,6 @@
 		<!--#########################################################################-->
 		<joint name="yaw_pitch_joint" type="continuous">
+			<origin xyz="0 0 0" rpy="0 0 ${initial_pitch_angle}" />
 			<axis xyz="0 0 1" />
-			<origin xyz="0 0 0" rpy="0 0 ${initial_pitch_angle}" />
 			<limit lower="${-M_PI/180*25}" upper="${M_PI/180*25}" effort="100000" velocity="100000" />
 			<parent link="yaw_link" />
@@ -95,6 +95,6 @@
 		<!--#########################################################################-->
 		<joint name="pitch_roll_joint" type="continuous">
-			<axis xyz="0 1 0" />
 			<origin xyz="${pitch_length + child_offset} ${-0.08*biped} 0" rpy="${-M_PI/2*biped} ${-M_PI/2 + M_PI/2*biped} ${-M_PI/2 + M_PI/2*biped + child_pitch}" />
+			<axis xyz="${biped} ${1-biped} 0" />
 			<parent link="pitch_link" />
 			<child link="${child_link}"/>
