Commit message: Split atrias20 into multiple files.
git-svn-id: https://atrias.googlecode.com/svn/trunk@818 a504bc44-2baa-4cb8-4136-ba805e94d278

File: drl-sim/atrias_sim/robots/atrias20_leg.urdf.xacro (robot description, xacro)
@@ -40,12 +40,12 @@
 	<property name="leg_damping" value="0" />
 	<property name="leg_friction" value="0" />
-	<!-- macro name used to insert this entire file into the header file when parsed by xacro -->
-	<xacro:macro name="atrias_leg" params="bodyLink">
+	<!-- macro to use in the header file when parsed by xacro -->
+	<xacro:macro name="atrias_leg" params="hip_link *origin">
 		<!--#########################################################################-->
 		<!--								Body                                     -->
 		<!--#########################################################################-->
-		<link name="${bodyLink}">
-			<inertial>
-				<origin xyz="0 0 0.002" />
+		<link name="${hip_link}">
+			<inertial>
+				<insert_block name="origin" />
 				<mass value="${body_mass}" />
 				<inertia ixx="0.0932" ixy="0.0044" ixz="-0.0019"
@@ -66,5 +66,5 @@
 			</collision>
 		</link>
-		<gazebo reference="${bodyLink}">
+		<gazebo reference="${hip_link}">
 			<material>Gazebo/BumpyMetal</material>
 		</gazebo>
@@ -75,5 +75,5 @@
 			<axis xyz="0 1 0" />
 			<origin xyz="0 0 0" rpy="0 0 0" />
-			<parent link="${bodyLink}" />
+			<parent link="${hip_link}" />
 			<child link="thighMotor_link" />
 			<limit lower="${-M_PI/4-0.3054}" upper="${-M_PI/4+2.3562}" effort="10000000000000" velocity="100000000000000" />
@@ -119,5 +119,5 @@
 			<axis xyz="0 1 0" />
 			<origin xyz="0 0 0" rpy="0 0 0" />
-			<parent link="${bodyLink}" />
+			<parent link="${hip_link}" />
 			<child link="shinMotor_link"/>
 			<limit lower="${-5*M_PI/4+2.8362}" upper="${-5*M_PI/4+5.4978}" effort="10000000000000" velocity="100000000000000" />
@@ -163,5 +163,5 @@
 			<axis xyz="0 1 0" />
 			<origin xyz="0 0 0" rpy="0 0 0" />
-			<parent link="${bodyLink}" />
+			<parent link="${hip_link}" />
 			<child link="thigh_link"/>
 			<!--limit lower="${-M_PI/4-0.6545}" upper="${-M_PI/4+2.7053}" effort="1000000000000" velocity="100000000000000" /-->
@@ -198,5 +198,5 @@
 			<axis xyz="0 1 0" />
 			<origin xyz="0 0 0" rpy="0 0 0" />
-			<parent link="${bodyLink}" />
+			<parent link="${hip_link}" />
 			<child link="shin_link"/>
 			<!--limit lower="${-5*M_PI/4+2.4871}" upper="${-5*M_PI/4+5.4978}" effort="100000000000" velocity="100000000000000" /-->

File: drl-sim/atrias_sim/robots/atrias20_planar_header.urdf.xacro (robot description, xacro)
@@ -14,8 +14,10 @@
 	<!-- get robot model macro -->
 	<include filename="atrias20_leg.urdf.xacro" />
-	<include filename="atrias20_planar_constraint.urdf.xacro" />
+	<include filename="planar_constraint.urdf.xacro" />
 	<!-- constrains and builds the atrias leg model -->
-	<xacro:atrias_planar_constraint attachmentLink="leg_body_link" />
-	<xacro:atrias_leg bodyLink="leg_body_link" />
+	<xacro:planar_constraint child_attachment_link="leg_hip_link" />
+	<xacro:atrias_leg hip_link="leg_hip_link">
+		<origin xyz="0 0 0.002" />
+	</xacro:atrias_leg>
 	<!-- initializes the all-in-one controller with the correct link names, etc. -->
 	<gazebo>
@@ -23,5 +25,5 @@
 			<alwaysOn> true </alwaysOn>
 			<updateRate> 1000 </updateRate>
-			<bodyName> leg_body_link </bodyName>
+			<bodyName> leg_hip_link </bodyName>
 			<motorAName> thighMotor_link </motorAName>
 			<motorBName> shinMotor_link </motorBName>

File: drl-sim/atrias_sim/robots/planar_constraint.urdf.xacro (robot description, xacro)
@@ -1,5 +1,5 @@
 <?xml version="1.0"?>
-<!-- ATRIAS 2.0 Robot Model -->
-<!-- Adapted for ATRIAS 2.0 in Winter Term 2012 by Andrew Peekema and Matthew Rueben -->
+<!-- Planar Linkage -->
+<!-- Created for ATRIAS 2.0 in Winter Term 2012 by Andrew Peekema and Matthew Rueben -->
 <robot
 	xmlns:sensor="http://playerstage.sourceforge.net/gazebo/xmlschema/#sensor"
@@ -16,5 +16,5 @@
 	<property name="SQRT_2" value="1.41421356"/>
 	<!-- macro name used to insert this entire file into the header file when parsed by xacro -->
-	<xacro:macro name="atrias_planar_constraint" params="attachmentLink">
+	<xacro:macro name="planar_constraint" params="child_attachment_link">
 		<!--#########################################################################-->
 		<!--							Planar Motion								-->
@@ -56,5 +56,5 @@
 			<axis xyz="0 1 0" />
 			<parent link="body_no_twist_link" />
-			<child link="${attachmentLink}"/>
+			<child link="${child_attachment_link}"/>
 		</joint>
 	</xacro:macro>

Commit message: Boom template
git-svn-id: https://atrias.googlecode.com/svn/trunk@837 a504bc44-2baa-4cb8-4136-ba805e94d278

File: drl-sim/atrias_sim/robots/atrias20_leg.urdf.xacro (robot description, xacro)
@@ -312,6 +312,6 @@
 		<!--							Toe											-->
 		<!--#########################################################################-->
-		<joint name="lower_toe_joint" type="fixed">
-			<origin xyz="${-lower_length/SQRT_2} 0 ${-lower_length/SQRT_2}" rpy="0 0 0" />
+		<joint name="lower_toe_joint" type="continuous">
+			<axis xyz="1 0 0" />
 			<parent link="lower_link" />
 			<child link="toe_link"/>

Commit message: Controller working with friction
git-svn-id: https://atrias.googlecode.com/svn/trunk@933 a504bc44-2baa-4cb8-4136-ba805e94d278

File: drl-sim/atrias_sim/robots/atrias20_leg.urdf.xacro (robot description, xacro)
@@ -35,9 +35,7 @@
 	<property name="toe_mass" value="0.087" />
 	<!-- Spring/Damping Coefficients -->
-	<property name="spring_stiffness" value="1200" />			<!-- N*m/rad -->
-	<property name="motor_damping" value="${2*0.5*34.64}" />	<!-- 2*Zeta*sqrt(K) (Guessed Zeta)-->
-	<property name="motor_friction" value="10" />				<!-- Guess -->
-	<property name="leg_damping" value="0" />
-	<property name="leg_friction" value="0" />
+	<property name="spring_stiffness" value="1200" />	<!-- N*m/rad -->
+	<property name="motor_damping" value="500" />		<!-- N*m*s/rad -->
+	<property name="motor_friction" value="0.1" />		<!-- N*m -->
 	<!-- macro to use in the header file when parsed by xacro -->
 	<xacro:macro name="atrias_leg" params="hip_link suffix *origin *axis" >
@@ -69,15 +67,24 @@
 			<material>Gazebo/BumpyMetal</material>
 		</gazebo>
+<!--
+        <gazebo>
+            <controller:position_body name="position_body" plugin="libposition_body.so">
+                <alwaysOn> true </alwaysOn>
+                <updateRate> 10000 </updateRate>
+                <bodyName> ${hip_link}${suffix} </bodyName>
+            </controller:position_body>
+        </gazebo>
+-->
 		<!--#########################################################################-->
 		<!--								Thigh Motor                              -->
 		<!--#########################################################################-->
-		<joint name="hip_thighMotor_joint${suffix}" type="revolute">
-			<axis xyz="0 1 0" />
+		<joint name="hip_thighMotor_joint${suffix}" type="continuous">
+			<axis xyz="0 1 0" />
+			<dynamics damping="0.0" friction="1000" />
 			<origin xyz="0 0 0" rpy="0 0 0" />
 			<parent link="${hip_link}${suffix}" />
 			<child link="thighMotor_link${suffix}" />
-			<limit lower="${-M_PI/4-0.3054}" upper="${-M_PI/4+2.3562}" effort="1000000" velocity="1000000" />
-			<dynamics damping="${motor_damping}" friction="${motor_friction}" />
-		</joint>
+<!--			<limit lower="${-M_PI/4-0.3054}" upper="${-M_PI/4+2.3562}" effort="1000000" velocity="1000000" />
+-->		</joint>
 		<link name="thighMotor_link${suffix}">
 			<inertial>
@@ -105,4 +112,12 @@
 		</gazebo>
 		<gazebo>
+            <controller:joint_impedance name="thighDamping${suffix}" plugin="libjoint_impedance.so">
+                <alwaysOn> true </alwaysOn>
+                <updateRate> 10000 </updateRate>
+				<bodyName1> ${hip_link}${suffix} </bodyName1>
+				<bodyName2> thighMotor_link${suffix} </bodyName2>
+                <rotationalDamping> ${motor_damping} </rotationalDamping>
+                <rotationalFriction> ${motor_friction} </rotationalFriction>
+            </controller:joint_impedance>
 			<controller:spring name="thighSpring${suffix}" plugin="libspring.so">
 				<alwaysOn> true </alwaysOn>
@@ -116,12 +131,11 @@
 		<!--					Shin Motor                                           -->
 		<!--#########################################################################-->
-		<joint name="hip_shinMotor_joint${suffix}" type="revolute">
+		<joint name="hip_shinMotor_joint${suffix}" type="continuous">
 			<axis xyz="0 1 0" />
 			<origin xyz="0 0 0" rpy="0 0 0" />
 			<parent link="${hip_link}${suffix}" />
 			<child link="shinMotor_link${suffix}"/>
-			<limit lower="${-5*M_PI/4+2.8362}" upper="${-5*M_PI/4+5.4978}" effort="10000000000000" velocity="100000000000000" />
-			<dynamics damping="${motor_damping}" friction="${motor_friction}" />
-		</joint>
+<!--			<limit lower="${-5*M_PI/4+2.8362}" upper="${-5*M_PI/4+5.4978}" effort="10000000000000" velocity="100000000000000" />
+-->		</joint>
 		<link name="shinMotor_link${suffix}">
 			<inertial>
@@ -148,5 +162,13 @@
 			<material>Gazebo/Green</material>
 		</gazebo>
-		<gazebo>
+        <gazebo>
+            <controller:joint_impedance name="shinDamping${suffix}" plugin="libjoint_impedance.so">
+                <alwaysOn> true </alwaysOn>
+                <updateRate> 10000 </updateRate>
+				<bodyName1> ${hip_link}${suffix} </bodyName1>
+				<bodyName2> shinMotor_link${suffix} </bodyName2>
+                <rotationalDamping> ${motor_damping} </rotationalDamping>
+                <rotationalFriction> ${motor_friction} </rotationalFriction>
+            </controller:joint_impedance>
 			<controller:spring name="shinSpring${suffix}" plugin="libspring.so">
 				<alwaysOn> true </alwaysOn>
@@ -165,7 +187,6 @@
 			<parent link="${hip_link}${suffix}" />
 			<child link="thigh_link${suffix}"/>
-			<!--limit lower="${-M_PI/4-0.6545}" upper="${-M_PI/4+2.7053}" effort="1000000000000" velocity="100000000000000" /-->
-			<dynamics damping="${leg_damping}" friction="${leg_friction}" />
-		</joint>
+<!--			<limit lower="${-M_PI/4-0.6545}" upper="${-M_PI/4+2.7053}" effort="1000000000000" velocity="100000000000000" />
+-->		</joint>
 		<link name="thigh_link${suffix}">
 			<inertial>
@@ -200,7 +221,6 @@
 			<parent link="${hip_link}${suffix}" />
 			<child link="shin_link${suffix}"/>
-			<!--limit lower="${-5*M_PI/4+2.4871}" upper="${-5*M_PI/4+5.4978}" effort="100000000000" velocity="100000000000000" /-->
-			<dynamics damping="${leg_damping}" friction="${leg_friction}" />
-		</joint>
+<!--			<limit lower="${-5*M_PI/4+2.4871}" upper="${-5*M_PI/4+5.4978}" effort="100000000000" velocity="100000000000000" />
+-->		</joint>
 		<link name="shin_link${suffix}">
 			<inertial>
@@ -230,11 +250,10 @@
 		<!--								 Lower Link					 			-->
 		<!--#########################################################################-->
-		<joint name="thigh_lower_joint${suffix}" type="continuous">
+		<joint name="thigh_lower_joint${suffix}" type="revolute">
 			<axis xyz="0 1 0" />
 			<origin xyz="${thigh_length/SQRT_2} 0 ${-thigh_length/SQRT_2}" rpy="0 0 0" />
 			<parent link="thigh_link${suffix}" />
 			<child link="lower_link${suffix}"/>
-			<limit lower="${-M_PI/2}" upper="${M_PI/2}" effort="10000000000000" velocity="100000000000000" />
-			<dynamics damping="${leg_damping}" friction="${leg_friction}" />
+			<limit lower="${-M_PI/2+0.05}" upper="${M_PI/2}" effort="10000000000000" velocity="100000000000000" />
 		</joint>
 		<link name="lower_link${suffix}">
@@ -265,11 +284,10 @@
 		<!--								 Four Bar	 							-->
 		<!--#########################################################################-->
-		<joint name="shin_fourBar_joint${suffix}" type="continuous">
+		<joint name="shin_fourBar_joint${suffix}" type="revolute">
 			<axis xyz="0 1 0" />
 			<origin xyz="${-shin_length/SQRT_2} 0 ${-shin_length/SQRT_2}" rpy="0 0 0" />
 			<parent link="shin_link${suffix}" />
 			<child link="fourBar_link${suffix}"/>
-			<limit lower="${-M_PI/2}" upper="${M_PI/2}" effort="10000000000000" velocity="100000000000000" />
-			<dynamics damping="${leg_damping}" friction="${leg_friction}" />
+			<limit lower="${-M_PI/2+0.05}" upper="${M_PI/2}" effort="10000000000000" velocity="100000000000000" />
 		</joint>
 		<link name="fourBar_link${suffix}">
@@ -340,4 +358,8 @@
 		</link>
 		<gazebo reference="toe_link${suffix}">
+			<mu1 value="100.0" />
+			<mu2 value="100.0" />
+			<kp  value="1000000.0" />
+			<kd  value="1.0" />
 			<material>Gazebo/Red</material>
 		</gazebo>

File: drl-sim/atrias_sim/robots/boomTest.urdf.xacro (robot description, xacro)
@@ -129,4 +129,14 @@
 		</gazebo>
 		<gazebo>
+			<controller:joint_impedance name="pendulum_damping" plugin="libjoint_impedance.so">
+				<alwaysOn> true </alwaysOn>
+				<updateRate> 10000 </updateRate>
+				<bodyName1> upright_link </bodyName1>
+				<bodyName2> pendulum_link </bodyName2>
+				<rotationalDamping> 0 </rotationalDamping>
+				<rotationalFriction> 0.01 </rotationalFriction>
+			</controller:joint_impedance>
+		</gazebo>
+		<gazebo>
 			<controller:spring name="pendulum_spring" plugin="libspring.so">
 				<alwaysOn> true </alwaysOn>

File: drl-sim/atrias_sim/robots/planar_constraint.urdf.xacro (robot description, xacro)
@@ -21,5 +21,5 @@
 		<!--#########################################################################-->
 		<link name="world" />
-		<joint name="world_joint" type="continuous">
+		<joint name="world_joint" type="fixed">
 			<origin xyz="0 0 0" rpy="0 0 0" />
 			<axis xyz="0 1 0" />
@@ -36,5 +36,5 @@
 			</inertial>
 		</link>
-		<joint name="planar_joint" type="prismatic">
+		<joint name="planar_joint" type="fixed">
 			<origin xyz="0 0 1.5" rpy="0 0 0" />
 			<axis xyz="0 0 1" />

Commit message: Modifications for controller testing
git-svn-id: https://atrias.googlecode.com/svn/trunk@939 a504bc44-2baa-4cb8-4136-ba805e94d278

File: drl-sim/atrias_sim/robots/atrias20_leg.urdf.xacro (robot description, xacro)
@@ -36,6 +36,6 @@
 	<!-- Spring/Damping Coefficients -->
 	<property name="spring_stiffness" value="1200" />	<!-- N*m/rad -->
-	<property name="motor_damping" value="500" />		<!-- N*m*s/rad -->
-	<property name="motor_friction" value="0.1" />		<!-- N*m -->
+	<property name="motor_damping" value="10" />		<!-- N*m*s/rad -->
+	<property name="motor_friction" value="10" />		<!-- N*m -->
 	<!-- macro to use in the header file when parsed by xacro -->
 	<xacro:macro name="atrias_leg" params="hip_link suffix *origin *axis" >
@@ -67,5 +67,4 @@
 			<material>Gazebo/BumpyMetal</material>
 		</gazebo>
-<!--
         <gazebo>
             <controller:position_body name="position_body" plugin="libposition_body.so">
@@ -75,5 +74,4 @@
             </controller:position_body>
         </gazebo>
--->
 		<!--#########################################################################-->
 		<!--								Thigh Motor                              -->
@@ -81,5 +79,4 @@
 		<joint name="hip_thighMotor_joint${suffix}" type="continuous">
 			<axis xyz="0 1 0" />
-			<dynamics damping="0.0" friction="1000" />
 			<origin xyz="0 0 0" rpy="0 0 0" />
 			<parent link="${hip_link}${suffix}" />

File: drl-sim/atrias_sim/robots/planar_constraint.urdf.xacro (robot description, xacro)
@@ -21,5 +21,5 @@
 		<!--#########################################################################-->
 		<link name="world" />
-		<joint name="world_joint" type="fixed">
+		<joint name="world_joint" type="continuous">
 			<origin xyz="0 0 0" rpy="0 0 0" />
 			<axis xyz="0 1 0" />
@@ -36,5 +36,5 @@
 			</inertial>
 		</link>
-		<joint name="planar_joint" type="fixed">
+		<joint name="planar_joint" type="prismatic">
 			<origin xyz="0 0 1.5" rpy="0 0 0" />
 			<axis xyz="0 0 1" />
