Commit message: Added a toe
git-svn-id: https://atrias.googlecode.com/svn/trunk@1016 a504bc44-2baa-4cb8-4136-ba805e94d278

File: drl-sim/atrias_sim/robots/inverted_pendulum_toe.urdf.xacro (robot description, xacro)
@@ -14,30 +14,37 @@
 	<property name="M_PI" value="3.14159"/>
 	<property name="SQRT_2" value="1.41421356"/>
-	<!--#########################################################################-->
-	<!--							Point Mass                                   -->
-	<!--#########################################################################-->
-	<link name="toe">
-		<inertial>
-			<origin xyz="0 0 0" rpy="0 0 0" />
-			<mass value="0.0001" />
-			<inertia ixx="0.001" ixy="0.0" ixz="0.0"
-					 iyy="0.0001" iyz="0.0"
-				     izz="0.0001" />
-		</inertial>
-		<visual>
-			<origin xyz="0 0 0" rpy="0 0 0" />
-			<geometry>
-			  <sphere radius="0.05" />
-			</geometry>
-		</visual>
-		<collision>
-			<origin xyz="0 0 0" rpy="0 0 0" />
-			<geometry>
-			  <sphere radius="0.05" />
-			</geometry>
-		</collision>
-	</link>
-	<gazebo reference="pointMass">
-		<material>Gazebo/Red</material>
-	</gazebo>
+    <xacro:macro name="invertedPendulumToe" params="toeName massName" >
+    	<!--#########################################################################-->
+    	<!--							Toe                                          -->
+    	<!--#########################################################################-->
+        <joint name="free_joint" type="floating">
+           <origin xyz="0 0 -0.9" rpy="0 0 0" />
+           <parent link="${massName}" />
+           <child link="${toeName}" />
+        </joint>
+    	<link name="${toeName}">
+    		<inertial>
+    			<origin xyz="0 0 0" rpy="0 0 0" />
+    			<mass value="0.0001" />
+    			<inertia ixx="0.001" ixy="0.0" ixz="0.0"
+    					 iyy="0.0001" iyz="0.0"
+    				     izz="0.0001" />
+    		</inertial>
+    		<visual>
+    			<origin xyz="0 0 0" rpy="0 0 0" />
+    			<geometry>
+    			  <sphere radius="0.05" />
+    			</geometry>
+    		</visual>
+    		<collision>
+    			<origin xyz="0 0 0" rpy="0 0 0" />
+    			<geometry>
+    			  <sphere radius="0.05" />
+    			</geometry>
+    		</collision>
+    	</link>
+    	<gazebo reference="${toeName}">
+    		<material>Gazebo/Red</material>
+    	</gazebo>
+    </xacro:macro>
 </robot>

Commit message: Added inverted pendulum with toe at proper heights
git-svn-id: https://atrias.googlecode.com/svn/trunk@1032 a504bc44-2baa-4cb8-4136-ba805e94d278

File: drl-sim/atrias_sim/robots/inverted_pendulum_toe.urdf.xacro (robot description, xacro)
@@ -19,5 +19,5 @@
     	<!--#########################################################################-->
         <joint name="free_joint" type="floating">
-           <origin xyz="0 0 -0.9" rpy="0 0 0" />
+           <origin xyz="0 0 -0.959" rpy="0 0 0" />
            <parent link="${massName}" />
            <child link="${toeName}" />

File: drl-sim/atrias_sim/robots/inverted_pendulum_with_toe_header.urdf.xacro (robot description, xacro)
@@ -20,10 +20,10 @@
 	<!-- initialize the controller -->
     <gazebo>
-        <controller:invertedPendulum name="Inverted_Pendulum" plugin="libinvertedPendulumWithToe.so">
+        <controller:invertedPendulumWithToe name="Inverted_Pendulum_With_Toe" plugin="libinvertedPendulumWithToe.so">
             <alwaysOn> true </alwaysOn>
             <updateRate> 10000 </updateRate>
             <bodyName1> pointMass </bodyName1>
             <bodyName2> toe </bodyName2>
-        </controller:invertedPendulum>
+        </controller:invertedPendulumWithToe>
     </gazebo>
 </robot>

Commit message: Made it work
git-svn-id: https://atrias.googlecode.com/svn/trunk@1100 a504bc44-2baa-4cb8-4136-ba805e94d278

File: drl-sim/atrias_sim/robots/inverted_pendulum_toe.urdf.xacro (robot description, xacro)
@@ -19,5 +19,5 @@
     	<!--#########################################################################-->
         <joint name="free_joint" type="floating">
-           <origin xyz="0 0 -0.959" rpy="0 0 0" />
+           <origin xyz="0 0 -0.909" rpy="0 0 0" />
            <parent link="${massName}" />
            <child link="${toeName}" />

Commit message: Delete old drl-sim and copy over drl-sim from newgui branch. This is the wrong way to merge, but there are too many changes to keep track of, and Subversion probably can't help us here.
git-svn-id: https://atrias.googlecode.com/svn/trunk@1388 a504bc44-2baa-4cb8-4136-ba805e94d278

File: drl-sim/atrias_sim/robots/inverted_pendulum_toe.urdf.xacro (robot description, xacro)
@@ -19,5 +19,5 @@
     	<!--#########################################################################-->
         <joint name="free_joint" type="floating">
-           <origin xyz="0 0 -0.909" rpy="0 0 0" />
+           <origin xyz="0 0 -0.959" rpy="0 0 0" />
            <parent link="${massName}" />
            <child link="${toeName}" />
